Commit message: delete build install log errados

File: novamob_nav2_gz/src/description/novamob_description.urdf (robot description, URDF)
Before this commit: robot novamob, 6 links, 5 joints
Links:
- link base_link: geometry collision box size=${base_length} ${base_width} ${base_height}; visual mesh filename=file://$(find novamob_nav2_gz)/meshes/novamob_no_wheels_cen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 scale=0.001 0.001 0.001

File: scout_description/urdf/scout_v2/scout_v2.xacro (robot description, xacro)
@@ -116,5 +116,5 @@
         <parent link="base_link"/>
         <child link="imu_link"/>
-        <origin xyz="0.0 0 0.01"/>
+        <origin xyz="0.0 0 0.0"/>
     </joint>
     <gazebo reference="imu_link">
