Commit message: Continuação trailer scout

File: novamob_nav2_gz/src/description/trailer_example.urdf (robot description, URDF)
Before this commit: robot car_trailer_robot, 3 links, 2 joints
Links:
- link car_base: geometry collision box size=1.3 2 0.1; visual box size=1.3 2 1

File: scout_nav2_gz/urdf/scout_v2/scout_v2_trailer.xacro (robot description, xacro)
@@ -17,9 +17,12 @@
     <xacro:property name="wheel_radius" value="1.6459e-01" />
     <xacro:property name="wheel_mass" value="0.6"/>
+    <xacro:property name="trailer_wheel_length" value="0.045" />
+    <xacro:property name="trailer_wheel_radius" value="0.06" />
+    <xacro:property name="trailer_wheel_mass" value="0.6"/>
     <xacro:property name="connector_length" value="0.15"/>
     <xacro:property name="connector_width" value="0.015"/>
     <xacro:property name="connector_height" value="0.015"/>
-    <xacro:property name="trailer_length" value="${base_x_size}"/>
-    <xacro:property name="trailer_width" value="${base_y_size}"/>
+    <xacro:property name="trailer_length" value="0.55"/>
+    <xacro:property name="trailer_width" value="0.4"/>
     <xacro:property name="trailer_height" value="${base_z_size}"/>
     <!-- Define inertial property macros  -->
@@ -112,5 +115,5 @@
       <visual>
         <geometry>
-          <cylinder radius="${wheel_radius}" length="${wheel_length}"/>
+          <cylinder radius="${trailer_wheel_radius}" length="${trailer_wheel_length}"/>
         </geometry>
         <origin xyz="0 0 0" rpy="${pi/2} ${pi/2} 0"/>
@@ -121,14 +124,14 @@
       <collision>
         <geometry>
-          <cylinder radius="${wheel_radius}" length="${wheel_length}"/>
+          <cylinder radius="${trailer_wheel_radius}" length="${trailer_wheel_length}"/>
         </geometry>
         <origin xyz="0 0 0" rpy="${pi/2} ${pi/2} 0"/>
       </collision>
-      <xacro:cylinder_inertia m="${wheel_mass}" r="${wheel_radius}" h="${wheel_length}"/>
+      <xacro:cylinder_inertia m="${trailer_wheel_mass}" r="${trailer_wheel_radius}" h="${trailer_wheel_length}"/>
     </link>
     <joint name="${prefix}_joint" type="continuous">
       <parent link="trailer_link"/>
       <child link="${prefix}_link"/>
-      <origin xyz="${x_reflect * wheel_offset} ${y_reflect * (trailer_width / 2 + wheel_length / 2)} ${-trailer_height / 2}" rpy="0 0 0"/>
+      <origin xyz="${x_reflect * wheel_offset} ${y_reflect * (trailer_width / 2 + trailer_wheel_length / 2)} ${-trailer_height / 2}" rpy="0 0 0"/>
       <axis xyz="0 1 0"/>
     </joint>
@@ -157,5 +160,5 @@
     <parent link="base_link"/>
     <child link="trailer_connector_link"/>
-    <origin xyz="${(-base_x_size/2)} 0 ${(base_z_size/2)} " rpy="0 0 0"/>
+    <origin xyz="${(-base_x_size/2)} 0 -0.065 " rpy="0 0 0"/>
     <axis xyz="0 0 1"/>
     <limit effort="100" velocity="2.0" lower="${-pi/4}" upper="${pi/4}"/>
@@ -193,5 +196,5 @@
   <xacro:trailer_wheel prefix="trailer_wheel_rf" x_reflect="1" y_reflect="-1" wheel_offset="${trailer_length / 4}"/>
   <xacro:trailer_wheel prefix="trailer_wheel_rr" x_reflect="-1" y_reflect="-1" wheel_offset="${trailer_length / 4}"/>
-    <!-- IMU -->
+  <!-- IMU -->
   <link name="imu_link">
     <visual>
