Commit message: Further trailer testing

File: novamob_nav2_gz/src/description/novamob_trailer_description.urdf (robot description, URDF)
Before this commit: robot novamob, 3 links, 2 joints
Joints:
- joint car_trailer_connector_joint: axis 0 1 1 -> 1 1 0

Commit message: Trailer for novamob 90% done

File: novamob_nav2_gz/src/description/novamob_trailer_description.urdf (robot description, URDF)
Before this commit: robot novamob, 3 links, 2 joints
Links:
- removed link trailer_connector_base
- added link camera_frame
- added link camera_link, mass 0.135; collision box size=0.030 0.124 0.030; visual box size=0.030 0.124 0.030
- added link imu_link; collision box size=0.01 0.01 0.01; visual box size=0.01 0.01 0.01
- added link lidar_link, mass 0.125; collision cylinder length=0.0275 radius=0.0254; visual cylinder length=0.0275 radius=0.0254
- added link trailer_connector_link; collision box size=${connector_width} ${connector_length} ${connector_height}; visual box size=${connector_width} ${connector_length} ${connector_height}
- added link trailer_link; collision box size=${trailer_length} ${trailer_width} ${trailer_height}; visual box size=${trailer_length} ${trailer_width} ${trailer_height}
Joints:
- removed joint car_trailer_connector_joint
- added joint camera_frame_joint: type fixed, parent camera_link, child camera_frame, origin xyz=0 0 0 rpy=${-pi/2} 0 ${-pi/2}
- added joint camera_joint: type fixed, parent base_link, child camera_link, origin xyz=0.09 0 ${platform_1_height + (0.022 / 2)} rpy=0 0 0
- added joint imu_joint: type fixed, parent base_link, child imu_link, origin xyz=0.0 0 0.01
- added joint lidar_joint: type fixed, parent base_link, child lidar_link, origin xyz=0 0 ${base_height + (0.0275/2)} rpy=0 0 0
- added joint trailer_connector_joint: type revolute, parent base_link, child trailer_connector_link, origin xyz=${(-base_length/2)} 0.0 ${platform_1_height}  rpy=0 0 0, axis 0 0 1, limit lower=${-pi/4} upper=${pi/4} effort=1000 velocity=2.0
- added joint trailer_joint: type fixed, parent trailer_connector_link, child trailer_link, origin xyz=${-((base_length/2) + connector_length)} 0 0 rpy=0 0 0, axis 0 0 1, limit lower=-3.14159 upper=3.14159 effort=1000 velocity=1

File: novamob_nav2_gz/src/description/trailer_example.urdf (robot description, URDF)
Before this commit: robot car_trailer_robot, 3 links, 2 joints
Links:
- link car_base: geometry collision box size=1.3 2 0.1; visual box size=${base_length} ${base_width} ${base_height}

Commit message: Small fix to trailers

File: novamob_nav2_gz/src/description/novamob_trailer_description.urdf (robot description, URDF)
Before this commit: robot novamob, 8 links, 7 joints
Joints:
- joint trailer_joint: origin xyz=${-((base_length/2) + connector_length)} 0 0 rpy=0 0 0 -> xyz=${-((trailer_length/2) + connector_length)} 0 0 rpy=0 0 0

File: scout_nav2_gz/urdf/scout_v2/scout_v2_trailer.xacro (robot description, xacro)
@@ -187,5 +187,5 @@
     <parent link="trailer_connector_link"/>
     <child link="trailer_link"/>
-    <origin xyz="${-((base_x_size/2) + connector_length)} 0 0" rpy="0 0 0"/>
+    <origin xyz="${-((trailer_length/2) + connector_length)} 0 0" rpy="0 0 0"/>
     <axis xyz="0 0 1"/>
     <limit effort="100" lower="-3.14159" upper="3.14159" velocity="1"/>
