Commit message: Added joint_state_publisher_gui to launch file (?)

File: novamob_description/src/description/novamob_trailer_description.urdf (robot description, URDF)
Before this commit: robot novamob, 8 links, 7 joints
Links:
- removed link camera_frame
- added link camera_depth_frame
- link base_link: geometry collision box size=${base_length} ${base_width} ${base_height}; visual mesh filename=file://$(find novamob_description)/meshes/novamob_no_wheels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 scale=0.001 0.001 0.001
Joints:
- removed joint camera_frame_joint
- added joint camera_depth_joint: type fixed, parent camera_link, child camera_depth_frame, origin xyz=0 0 0 rpy=${-pi/2} 0 ${-pi/2}

Commit message: Small changes to trailer

File: novamob_description/src/description/novamob_trailer_description.urdf (robot description, URDF)
Before this commit: robot novamob, 8 links, 7 joints
Joints:
- joint trailer_connector_joint: limit lower=${-pi/4} upper=${pi/4} effort=1000 velocity=2.0 -> lower=${-pi/4} upper=${pi/4} effort=100 velocity=2.0
- joint trailer_joint: limit lower=-3.14159 upper=3.14159 effort=1000 velocity=1 -> lower=-3.14159 upper=3.14159 effort=100 velocity=1

File: novamob_nav2_gz/src/description/novamob_trailer_description.urdf (robot description, URDF)
Before this commit: robot novamob, 8 links, 7 joints
Joints:
- joint trailer_connector_joint: limit lower=${-pi/4} upper=${pi/4} effort=1000 velocity=2.0 -> lower=${-pi/4} upper=${pi/4} effort=100 velocity=2.0
- joint trailer_joint: limit lower=-3.14159 upper=3.14159 effort=1000 velocity=1 -> lower=-3.14159 upper=3.14159 effort=100 velocity=1

Commit message: Changes to trailer_joint

File: novamob_description/src/description/novamob_trailer_description.urdf (robot description, URDF)
Before this commit: robot novamob, 8 links, 7 joints
Joints:
- joint trailer_joint: origin xyz=${-((base_length/2) + connector_length)} 0 0 rpy=0 0 0 -> xyz=${-(connector_length)} 0 0 rpy=0 0 0

File: novamob_nav2_gz/src/description/novamob_trailer_description.urdf (robot description, URDF)
Before this commit: robot novamob, 8 links, 7 joints
Joints:
- joint trailer_joint: origin xyz=${-((trailer_length/2) + connector_length)} 0 0 rpy=0 0 0 -> xyz=${-(connector_length)} 0 0 rpy=0 0 0
