Commit message: Changed scout's lidar and camera specs to match real world

File: scout_nav2_gz/urdf/scout_v2/scout_v2.xacro (robot description, xacro)
@@ -235,5 +235,5 @@
       <origin xyz="0 0 0" rpy="0 0 0"/>
       <geometry>
-        <cylinder radius="0.0254" length="0.0275"/>
+        <cylinder radius="0.06" length="0.086"/>
       </geometry>
     </collision>
@@ -241,5 +241,5 @@
       <origin xyz="0 0 0" rpy="0 0 0"/>
       <geometry>
-        <cylinder radius="0.0254" length="0.0275"/>
+        <cylinder radius="0.06" length="0.086"/>
       </geometry>
     </visual>
@@ -248,6 +248,7 @@
         <parent link="base_link"/>
         <child link="lidar_link"/>
-        <origin xyz="0.25 0 ${(base_z_size/2) + 0.02 + 0.0275}" rpy="0 0 0"/>
+        <origin xyz="0.25 0 ${(base_z_size/2) + 0.02 + 0.086}" rpy="0 0 0"/>
   </joint>
+  <!-- Based on the VLP 16 Lidar -->
   <gazebo reference="lidar_link">
     <sensor name="lidar" type="gpu_lidar">
@@ -256,18 +257,23 @@
       <always_on>true</always_on>
       <visualize>true</visualize>
-      <update_rate>5</update_rate>
+      <update_rate>20</update_rate>
       <lidar>
         <scan>
           <horizontal>
             <samples>360</samples>
-            <resolution>1.000000</resolution>
+            <resolution>0.1</resolution>
             <min_angle>0.000000</min_angle>
             <max_angle>6.280000</max_angle>
           </horizontal>
+          <vertical>
+            <samples>16</samples> <!-- VLP-16 specific -->
+            <min_angle>-0.261799</min_angle> <!-- -15° in radians -->
+            <max_angle>0.261799</max_angle> <!-- 15° in radians -->
+          </vertical>
         </scan>
         <range>
           <min>0.150000</min>
-          <max>12</max>
-          <resolution>0.015000</resolution>
+          <max>100</max>
+          <resolution>0.01</resolution>
         </range>
         <noise>
@@ -314,12 +320,13 @@
     <sensor name="robot_cam" type="camera">
       <camera>
-        <horizontal_fov>1.047</horizontal_fov>
+        <horizontal_fov>1.204</horizontal_fov>  <!-- Horizontal FOV 69° -->
+        <vertical_fov>0.73</vertical_fov> <!-- Vertical FOV 42° -->
         <image>
-          <width>320</width>
-          <height>240</height>
+          <width>1920</width>
+          <height>1080</height>
         </image>
         <clip>
-          <near>0.1</near>
-          <far>100</far>
+          <near>0.2</near>
+          <far>10</far>
         </clip>
       </camera>
@@ -330,4 +337,23 @@
       <enable_metrics>true</enable_metrics>
     </sensor>
+    <sensor name="depth_camera1" type="depth_camera">
+      <update_rate>90</update_rate>
+      <topic>depth_camera</topic>
+      <visualize>true</visualize>
+      <alwaysOn>true</alwaysOn>
+      <camera>
+        <horizontal_fov>1.518</horizontal_fov>  <!-- Horizontal FOV 87° -->
+        <vertical_fov>1.01</vertical_fov> <!-- Vertical FOV 58° -->
+        <image>
+          <width>1280</width>
+          <height>720</height>
+          <format>R_FLOAT32</format>
+        </image>
+        <clip>
+          <near>0.2</near>
+          <far>10</far>
+        </clip>
+      </camera>
+    </sensor>
   </gazebo>
 </robot>

Commit message: Added stands for lidar and camera, aligning with the real scout

File: scout_nav2_gz/urdf/scout_v2/scout_v2.xacro (robot description, xacro)
@@ -99,4 +99,52 @@
         <origin xyz="${-wheelbase/2} ${-track/2} ${wheel_vertical_offset}" rpy="3.14 0 0" />
     </xacro:scout_wheel_type2>
+  <!-- Camera stand box -->
+  <link name="camera_stand_link">
+      <visual>
+          <origin xyz="0 0 0" rpy="0 0 0"/>
+          <geometry>
+              <box size="0.15 0.15 0.01"/> <!-- Adjust size as needed -->
+          </geometry>
+          <material name="Gray">
+              <color rgba="0.5 0.5 0.5 1.0"/>
+          </material>
+      </visual>
+      <collision>
+          <origin xyz="0 0 0" rpy="0 0 0"/>
+          <geometry>
+              <box size="0.15 0.15 0.01"/> <!-- Same size for collision -->
+          </geometry>
+      </collision>
+      <xacro:box_inertia m="0.1" w="0.1" d="0.1" h="0.1"/>
+  </link>
+  <joint name="camera_stand_joint" type="fixed">
+      <parent link="base_link"/>
+      <child link="camera_stand_link"/>
+      <origin xyz="0.24 0 ${(base_z_size/2) + 0.0127}" rpy="0 0 0"/>
+  </joint>
+  <!-- Lidar stand box -->
+  <link name="lidar_stand_link">
+      <visual>
+          <origin xyz="0 0 0" rpy="0 0 0"/>
+          <geometry>
+              <box size="0.1 0.15 0.04"/> <!-- Adjust size as needed -->
+          </geometry>
+          <material name="Gray">
+              <color rgba="0.5 0.5 0.5 1.0"/>
+          </material>
+      </visual>
+      <collision>
+          <origin xyz="0 0 0" rpy="0 0 0"/>
+          <geometry>
+              <box size="0.1 0.15 0.04"/> <!-- Same size for collision -->
+          </geometry>
+      </collision>
+      <xacro:box_inertia m="0.1" w="0.1" d="0.1" h="0.1"/>
+  </link>
+  <joint name="lidar_stand_joint" type="fixed">
+      <parent link="camera_stand_link"/>
+      <child link="lidar_stand_link"/>
+      <origin xyz="-0.01 0 0.025" rpy="0 0 0"/>
+  </joint>
     <!-- IMU -->
   <link name="imu_link">
@@ -307,7 +355,7 @@
   </link>
   <joint name="camera_joint" type="fixed">
-    <parent link="base_link"/>
+    <parent link="camera_stand_link"/>
     <child link="camera_link"/>
-    <origin xyz="0.25 0 ${(base_z_size/2) + 0.02}" rpy="0 0 0"/>
+    <origin xyz="0.06 0 0.02" rpy="0 0 0"/>
   </joint>
   <link name="camera_frame"/>

File: scout_nav2_gz/urdf/scout_v2/scout_v2_trailer.xacro (robot description, xacro)
@@ -109,4 +109,52 @@
         <origin xyz="${-wheelbase/2} ${-track/2} ${wheel_vertical_offset}" rpy="3.14 0 0" />
     </xacro:scout_wheel_type2>
+  <!-- Camera stand box -->
+  <link name="camera_stand_link">
+      <visual>
+          <origin xyz="0 0 0" rpy="0 0 0"/>
+          <geometry>
+              <box size="0.15 0.15 0.01"/> <!-- Adjust size as needed -->
+          </geometry>
+          <material name="Gray">
+              <color rgba="0.5 0.5 0.5 1.0"/>
+          </material>
+      </visual>
+      <collision>
+          <origin xyz="0 0 0" rpy="0 0 0"/>
+          <geometry>
+              <box size="0.15 0.15 0.01"/> <!-- Same size for collision -->
+          </geometry>
+      </collision>
+      <xacro:box_inertia m="0.1" w="0.1" d="0.1" h="0.1"/>
+  </link>
+  <joint name="camera_stand_joint" type="fixed">
+      <parent link="base_link"/>
+      <child link="camera_stand_link"/>
+      <origin xyz="0.24 0 ${(base_z_size/2) + 0.0127}" rpy="0 0 0"/>
+  </joint>
+  <!-- Lidar stand box -->
+  <link name="lidar_stand_link">
+      <visual>
+          <origin xyz="0 0 0" rpy="0 0 0"/>
+          <geometry>
+              <box size="0.1 0.15 0.04"/> <!-- Adjust size as needed -->
+          </geometry>
+          <material name="Gray">
+              <color rgba="0.5 0.5 0.5 1.0"/>
+          </material>
+      </visual>
+      <collision>
+          <origin xyz="0 0 0" rpy="0 0 0"/>
+          <geometry>
+              <box size="0.1 0.15 0.04"/> <!-- Same size for collision -->
+          </geometry>
+      </collision>
+      <xacro:box_inertia m="0.1" w="0.1" d="0.1" h="0.1"/>
+  </link>
+  <joint name="lidar_stand_joint" type="fixed">
+      <parent link="camera_stand_link"/>
+      <child link="lidar_stand_link"/>
+      <origin xyz="-0.01 0 0.025" rpy="0 0 0"/>
+  </joint>
   <!--                TRAILER             -->
   <!-- Trailer wheel macro -->
@@ -359,5 +407,5 @@
           <horizontal>
             <samples>360</samples>
-            <resolution>0.1</resolution>
+            <resolution>1.000000</resolution>
             <min_angle>0.000000</min_angle>
             <max_angle>6.280000</max_angle>
@@ -404,7 +452,7 @@
   </link>
   <joint name="camera_joint" type="fixed">
-    <parent link="base_link"/>
+    <parent link="camera_stand_link"/>
     <child link="camera_link"/>
-    <origin xyz="0.25 0 ${(base_z_size/2) + 0.02}" rpy="0 0 0"/>
+    <origin xyz="0.06 0 0.02" rpy="0 0 0"/>
   </joint>
   <link name="camera_frame"/>

Commit message: Added gps sensor  to start testing

File: scout_nav2_gz/urdf/scout_v2/scout_v2.xacro (robot description, xacro)
@@ -405,3 +405,32 @@
     </sensor>
   </gazebo>
+<!-- GPS Link -->
+<link name="gps_link">
+  <visual>
+    <geometry>
+      <box size="0.01 0.01 0.01"/>
+    </geometry>
+  </visual>
+  <collision>
+    <geometry>
+      <box size="0.01 0.01 0.01"/>
+    </geometry>
+  </collision>
+  <xacro:box_inertia m="0.1" w="0.1" d="0.1" h="0.1"/>
+</link>
+<!-- Joint for GPS -->
+<joint name="gps_joint" type="fixed">
+  <parent link="base_link"/>
+  <child link="gps_link"/>
+  <origin xyz="0.0 0 0.1"/> <!-- Adjust position as needed -->
+</joint>
+<gazebo reference="gps_link">
+  <sensor name="gps_sensor" type="navsat">
+    <plugin filename="ignition-gazebo-navsat-system" name="ignition::gazebo::systems::NavSat">
+    </plugin>
+    <topic>navsat</topic>
+    <always_on>true</always_on>
+    <update_rate>1</update_rate>
+  </sensor>
+</gazebo>
 </robot>

Commit message: Fixed lidar positionin scout

File: scout_nav2_gz/urdf/scout_v2/scout_v2.xacro (robot description, xacro)
@@ -296,5 +296,5 @@
         <parent link="base_link"/>
         <child link="lidar_link"/>
-        <origin xyz="0.25 0 ${(base_z_size/2) + 0.02 + 0.086}" rpy="0 0 0"/>
+        <origin xyz="0.25 0 ${(base_z_size/2) + 0.0127 + 0.025 + 0.02 + (0.086/2)}" rpy="0 0 0"/>
   </joint>
   <!-- Based on the VLP 16 Lidar -->

File: scout_nav2_gz/urdf/scout_v2/scout_v2_trailer.xacro (robot description, xacro)
@@ -393,5 +393,5 @@
         <parent link="base_link"/>
         <child link="lidar_link"/>
-        <origin xyz="0.25 0 ${(base_z_size/2) + 0.02 + 0.086}" rpy="0 0 0"/>
+        <origin xyz="0.25 0 ${(base_z_size/2) + 0.0127 + 0.025 + 0.02 + (0.086/2)}" rpy="0 0 0"/>
   </joint>
   <!-- Based on the VLP 16 Lidar -->
