Commit message: Fixed scout wheels

File: scout_description/urdf/scout_v2/scout_v2.xacro (robot description, xacro)
@@ -122,5 +122,5 @@
         <plugin filename="libgazebo_ros_imu_sensor.so" name="imu_plugin">
             <ros>
-            <namespace>/demo</namespace>
+            <!-- <namespace>/demo</namespace> -->
             <remapping>~/out:=imu</remapping>
             </ros>
@@ -189,7 +189,7 @@
     <gazebo>
         <plugin name='diff_drive' filename='libgazebo_ros_diff_drive.so'>
-        <ros>
+        <!-- <ros>
             <namespace>/demo</namespace>
-        </ros>
+        </ros> -->
         <num_wheel_pairs>2</num_wheel_pairs>
         <!--back wheels -->
@@ -205,7 +205,10 @@
         <wheel_diameter>${wheel_radius*2}</wheel_diameter>
         <!-- limits -->
-        <max_wheel_torque>20</max_wheel_torque>
+        <max_wheel_torque>1000</max_wheel_torque>
         <max_wheel_acceleration>1.0</max_wheel_acceleration>
         <updateRate>100</updateRate>
+        <covariance_x>0.000100</covariance_x>
+        <covariance_y>0.000100</covariance_y>
+        <covariance_yaw>0.010000</covariance_yaw>
         <!-- output -->
         <publish_odom>true</publish_odom>
@@ -216,4 +219,25 @@
         </plugin>
     </gazebo>
+<!--     <gazebo>
+        <plugin name="skid_steer_drive_controller" filename="libgazebo_ros_skid_steer_drive.so">
+            <updateRate>100.0</updateRate>
+            <robotNamespace></robotNamespace>
+            <leftFrontJoint>front_left_wheel</leftFrontJoint>
+            <rightFrontJoint>front_right_wheel</rightFrontJoint>
+            <leftRearJoint>rear_left_wheel</leftRearJoint>
+            <rightRearJoint>rear_right_wheel</rightRearJoint>
+            <wheelSeparation>4</wheelSeparation>
+            <wheelDiameter>0.32918</wheelDiameter>
+            <robotBaseFrame>base_link</robotBaseFrame>
+            <torque>1000</torque>
+            <commandTopic>cmd_vel</commandTopic>
+            <broadcastTF>true</broadcastTF>
+            <odometryTopic>odom</odometryTopic>
+            <odometryFrame>odom</odometryFrame>
+            <covariance_x>0.000100</covariance_x>
+            <covariance_y>0.000100</covariance_y>
+            <covariance_yaw>0.010000</covariance_yaw>
+        </plugin>
+    </gazebo> -->
     <!-- LIDAR -->
     <link name="lidar_link">
@@ -239,5 +263,5 @@
         <parent link="base_link"/>
         <child link="lidar_link"/>
-        <origin xyz="0.25 0 ${(base_z_size/2) + 0.02 + 0.0275}" rpy="0 0 0"/>
+        <origin xyz="0.4 0 ${(base_z_size/2) + 0.02 + 0.0275}" rpy="0 0 0"/>
     </joint>
     <gazebo reference="lidar_link">
@@ -300,5 +324,5 @@
         <parent link="base_link"/>
         <child link="camera_link"/>
-        <origin xyz="0.25 0 ${(base_z_size/2) + 0.02}" rpy="0 0 0"/>
+        <origin xyz="0.4 0 ${(base_z_size/2) + 0.02}" rpy="0 0 0"/>
     </joint>
     <link name="camera_depth_frame"/>

Commit message: Small fix to scout in gz classic

File: scout_description/urdf/scout_v2/scout_v2.xacro (robot description, xacro)
@@ -299,5 +299,5 @@
         </sensor>
     </gazebo>
-    <!-- Camera/Deph Sensor -->
+    <!-- Camera/Depth Sensor -->
     <link name="camera_link">
     <visual>

File: scout_description/urdf/scout_v2/scout_v2_trailer.xacro (robot description, xacro)
@@ -18,5 +18,5 @@
     <xacro:property name="wheel_mass" value="0.6"/>
     <xacro:property name="trailer_wheel_length" value="0.045" />
-    <xacro:property name="trailer_wheel_radius" value="0.06" />
+    <xacro:property name="trailer_wheel_radius" value="0.065" />
     <xacro:property name="trailer_wheel_mass" value="0.6"/>
     <xacro:property name="connector_length" value="0.15"/>
